File: Concepts/USB-to-UART/REV1/REV1.brd (EAGLE design)
At the start: 86.5 x 92.8 mm, 75 parts, among them IC1 FT4232HL, IC2 93LC56BT-I/OT, IC3 74HC595D, IC4 MAX3241EWI-T, IC5 MAX3241EWI-T, IC6 MAX3241EWI-T, IC7 MAX3241EWI-T, J1 USB-B-S-X-X-TH, J2 RJHSE-5384, J3 RJHSE-5384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

Commit message: Update REV1.brd
Routing:
- net DTX: track 70.4 -> 66.9 mm
- net +3V3: track 285.2 -> 286.1 mm
- net GND: vias 181 -> 180
Other:
- board text added: "OPT"
- board text added: "OPTIONAL"

Commit message: Update REV1.brd
Routing:
- net DTX: track 66.9 -> 69.2 mm
- net +3V3: track 286.1 -> 288.3 mm
- net DRX: track 100.1 -> 99.4 mm
- net TTL_TXD_A: track 41.1 -> 40.5 mm
- net LED_R4: track 7.31 -> 7.89 mm
- net TTL_TXD_A1: track 36.4 -> 36.9 mm
- net GND: track 38.1 -> 38.0 mm, vias 180 -> 179
